File: AS5048Encoder/AS5048 Encoder/AS5048 Encoder.sch (EAGLE design)
At the start: 6 parts, among them X1 SI-50170

Commit message: reroute and move around
Parts:
- added SV1: (no value), con-lstb:MA03-1
- added U$1: TERMINALBLOCK277-1667-ND, makesmith:TERMINALBLOCK277-1667-ND
Connections:
- new net PWR: SV1.2, U$1.2
- new net SERVO: SV1.1, X1.RCT
- net GND: now also SV1.3, U$1.1
Changed lines of the file:
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@@
 <part name="R1" library="eagle-ltspice" deviceset="R" device="" value="270"/>
 <part name="R2" library="eagle-ltspice" deviceset="R" device="" value="270"/>
+<part name="SV1" library="con-lstb" deviceset="MA03-1" device=""/>
+<part name="U$1" library="makesmith" deviceset="TERMINALBLOCK277-1667-ND" device=""/>
 </parts>
 <sheets>
@@
 <instance part="R1" gate="G$1" x="22.86" y="-15.24" rot="R90"/>
 <instance part="R2" gate="G$1" x="30.48" y="-15.24" rot="R90"/>
+<instance part="SV1" gate="G$1" x="45.72" y="45.72" rot="R270"/>
+<instance part="U$1" gate="G$1" x="66.04" y="43.18"/>
 </instances>
 <busses>
@@
 <label x="48.26" y="-20.32" size="1.778" layer="95"/>
 </segment>
+<segment>
+<pinref part="SV1" gate="G$1" pin="3"/>
+<wire x1="48.26" y1="38.1" x2="48.26" y2="35.56" width="0.1524" layer="91"/>
+<label x="48.26" y="30.48" size="1.778" layer="95" rot="R90"/>
+</segment>
+<segment>
+<label x="63.5" y="27.94" size="1.778" layer="95" rot="R90"/>
+<pinref part="U$1" gate="G$1" pin="1"/>
+<wire x1="63.5" y1="33.02" x2="63.5" y2="35.56" width="0.1524" layer="91"/>
+</segment>
 </net>
 <net name="VCC" class="0">
@@
 </segment>
 </net>
+<net name="SERVO" class="0">
+<segment>
+<pinref part="SV1" gate="G$1" pin="1"/>
+<wire x1="43.18" y1="38.1" x2="43.18" y2="35.56" width="0.1524" layer="91"/>
+<label x="43.18" y="27.94" size="1.778" layer="95" rot="R90"/>
+</segment>
+<segment>
+<pinref part="X1" gate="G$1" pin="RCT"/>
+<wire x1="55.88" y1="-2.54" x2="53.34" y2="-2.54" width="0.1524" layer="91"/>
+<label x="45.72" y="-2.54" size="1.778" layer="95"/>
+</segment>
+</net>
+<net name="PWR" class="0">
+<segment>
+<pinref part="SV1" gate="G$1" pin="2"/>
+<wire x1="45.72" y1="38.1" x2="45.72" y2="35.56" width="0.1524" layer="91"/>
+<label x="45.72" y="30.48" size="1.778" layer="95" rot="R90"/>
+</segment>
+<segment>
+<label x="71.12" y="27.94" size="1.778" layer="95" rot="R90"/>
+<pinref part="U$1" gate="G$1" pin="2"/>
+<wire x1="68.58" y1="33.02" x2="68.58" y2="35.56" width="0.1524" layer="91"/>
+</segment>
+</net>
